File: pcb/bizcard.kicad_sch (KiCad schematic)
At the start: 45 parts, among them J1 Conn_01x12_Female, J2 USB_C_ReceptacleUSB2.0, J3 Conn_ARM_JTAG_SWD_10, SW1 SW_Push, SW2 SW_Push, U1 AMS1117-3.3, U2 W25Q128JVS, U3 RP2040, Y1 12MHz

Commit message: fix schematic
Parts:
- C4, C5: value 27p -> 30p; LCSC C1557 -> C1570
Changed lines of the file:
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@@
       (effects (font (size 1.27 1.27)) (justify left))
     )
-    (property "Value" "27p" (id 1) (at 25.527 105.791 0)
+    (property "Value" "30p" (id 1) (at 25.527 105.791 0)
       (effects (font (size 1.27 1.27)) (justify left))
     )
@@
       (effects (font (size 1.27 1.27)) hide)
     )
-    (property "LCSC" "C1557" (id 4) (at 26.67 102.87 0)
+    (property "LCSC" "C1570" (id 4) (at 26.67 102.87 0)
       (effects (font (size 1.27 1.27)) hide)
     )
@@
       (effects (font (size 1.27 1.27)) (justify left))
     )
-    (property "Value" "27p" (id 1) (at 25.527 115.951 0)
+    (property "Value" "30p" (id 1) (at 25.527 115.951 0)
       (effects (font (size 1.27 1.27)) (justify left))
     )
@@
       (effects (font (size 1.27 1.27)) hide)
     )
-    (property "LCSC" "C1557" (id 4) (at 26.67 113.03 0)
+    (property "LCSC" "C1570" (id 4) (at 26.67 113.03 0)
       (effects (font (size 1.27 1.27)) hide)
     )
@@
       (effects (font (size 1.27 1.27)) (justify left))
     )
-    (property "Value" "12MHz" (id 1) (at 35.56 100.33 90)
+    (property "Value" "12MHz" (id 1) (at 39.37 100.33 90)
       (effects (font (size 1.27 1.27)) (justify left))
     )
@@
     )
     (path "/62dc79fe-cafa-403e-9613-995bf9a7d70b"
-      (reference "C4") (unit 1) (value "27p") (footprint "Capacitor_SMD:C_0402_1005Metric")
+      (reference "C4") (unit 1) (value "30p") (footprint "Capacitor_SMD:C_0402_1005Metric")
     )
     (path "/74e6db69-798d-468f-80af-963391df72a4"
-      (reference "C5") (unit 1) (value "27p") (footprint "Capacitor_SMD:C_0402_1005Metric")
+      (reference "C5") (unit 1) (value "30p") (footprint "Capacitor_SMD:C_0402_1005Metric")
     )
     (path "/8a977f34-a2fc-4574-8c85-433488616293"
